Commit message: Launch files

File: ros2_ws/src/my_robot_description/urdf/common_properties.xacro (robot description, xacro)
@@ -7,3 +7,30 @@
         <color rgba="0.25 0.25 0.25 1"/>
     </material>
+    <xacro:macro name="box_inertia" params="m x y z o_xyz o_rpy">
+        <inertial>
+            <mass value="${m}" />
+            <origin xyz="${o_xyz}" rpy="${o_rpy}"/>
+            <inertia ixx="${(m/12) * (y * y + z * z)}" ixy="0" ixz="0"
+                      iyy="${(m/12) * (x * x + z * z)}" iyz="0"
+                      izz="${(m/12) * (x * x + y * y)}" /> <!-- refer to wiki on intertial tensors/moments -->
+        </inertial>
+    </xacro:macro>
+    <xacro:macro name="cylinder_inertia" params="m r h o_xyz o_rpy">
+        <inertial>
+            <mass value="${m}" />
+            <origin xyz="${o_xyz}" rpy="${o_rpy}"/>
+            <inertia ixx="${(m/12) * (3 * r * r + h * h)}" ixy="0" ixz="0"
+                      iyy="${(m/12) * (3 * r * r + h * h)}" iyz="0"
+                      izz="${(m/2) * (r * r)}" /> <!-- refer to wiki on intertial tensors/moments -->
+        </inertial>
+    </xacro:macro>
+    <xacro:macro name="sphere_inertia" params="m r o_xyz o_rpy">
+        <inertial>
+            <mass value="${m}" />
+            <origin xyz="${o_xyz}" rpy="${o_rpy}"/>
+            <inertia ixx="${(2/5) * (m * r * r)}" ixy="0" ixz="0"
+                      iyy="${(2/5) * (m * r * r)}" iyz="0"
+                      izz="${(2/5) * (m * r * r)}" /> <!-- refer to wiki on intertial tensors/moments -->
+        </inertial>
+    </xacro:macro>
 </robot>

File: ros2_ws/src/my_robot_description/urdf/mobile_base.xacro (robot description, xacro)
@@ -15,4 +15,12 @@
                 <material name="grey" />
             </visual>
+            <xacro:cylinder_inertia m="5.0" r="${wheel_radius}" h="${wheel_length}"
+                            o_xyz="0 0 0" o_rpy="${pi / 2.0} 0 0"/>
+            <collision>
+                <geometry>
+                    <sphere radius="${wheel_radius}" />
+                </geometry>
+                <origin xyz="0 0 0" rpy="${pi / 2.0} 0 0" />
+            </collision>
         </link>
     </xacro:macro>
@@ -28,4 +36,12 @@
             <material name="green" />
         </visual>
+        <xacro:box_inertia m="5.0" x="${base_length}" y="${base_width}" z="${base_height}"
+                            o_xyz="0 0 ${base_height / 2.0}" o_rpy="0 0 0"/>
+         <collision>
+                <geometry>
+                    <box size="${base_length} ${base_width} ${base_height}" />
+                </geometry>
+                <origin xyz="0 0 ${base_height / 2.0}" rpy="0 0 0" />
+        </collision>
     </link>
     <link name="caster_wheel_link">
@@ -37,4 +53,12 @@
             <material name="grey" />
         </visual>
+        <xacro:sphere_inertia m="5.0" r="${wheel_radius / 2.0}"
+                            o_xyz="0 0 0" o_rpy="0 0 0" />
+        <collision>
+                <geometry>
+                    <sphere radius="${wheel_radius / 2.0}" />
+                </geometry>
+                <origin xyz="0 0 0" rpy="0 0 0" />
+        </collision>
     </link>
     <joint name="base_joint" type="fixed">

Commit message: Final

File: ros2_ws/src/my_robot_description/urdf/common_properties.xacro (robot description, xacro)
@@ -1,26 +1,32 @@
 <?xml version="1.0"?>
 <robot xmlns:xacro="http://www.ros.org/wiki/xacro">
-    <material name="green">
-        <color rgba="0 0.5 1 1"/>
+    <material name="blue">
+        <color rgba="0 0 0.5 1" />
     </material>
-        <material name="grey">
-        <color rgba="0.25 0.25 0.25 1"/>
+    <material name="grey">
+        <color rgba="0.5 0.5 0.5 1" />
+    </material>
+    <material name="orange">
+        <color rgba="1.0 0.5 0 1" />
+    </material>
+    <material name="yellow">
+        <color rgba="1.0 1.0 0 1" />
     </material>
     <xacro:macro name="box_inertia" params="m x y z o_xyz o_rpy">
         <inertial>
             <mass value="${m}" />
-            <origin xyz="${o_xyz}" rpy="${o_rpy}"/>
-            <inertia ixx="${(m/12) * (y * y + z * z)}" ixy="0" ixz="0"
-                      iyy="${(m/12) * (x * x + z * z)}" iyz="0"
-                      izz="${(m/12) * (x * x + y * y)}" /> <!-- refer to wiki on intertial tensors/moments -->
+            <origin xyz="${o_xyz}" rpy="${o_rpy}" />
+            <inertia ixx="${(m/12) * (y*y + z*z)}" ixy="0" ixz="0"
+                     iyy="${(m/12) * (x*x + z*z)}" iyz="0"
+                     izz="${(m/12) * (x*x + y*y)}" />
         </inertial>
     </xacro:macro>
-    <xacro:macro name="cylinder_inertia" params="m r h o_xyz o_rpy">
+    <xacro:macro name="cylinder_inertia" params="m r l o_xyz o_rpy">
         <inertial>
             <mass value="${m}" />
-            <origin xyz="${o_xyz}" rpy="${o_rpy}"/>
-            <inertia ixx="${(m/12) * (3 * r * r + h * h)}" ixy="0" ixz="0"
-                      iyy="${(m/12) * (3 * r * r + h * h)}" iyz="0"
-                      izz="${(m/2) * (r * r)}" /> <!-- refer to wiki on intertial tensors/moments -->
+            <origin xyz="${o_xyz}" rpy="${o_rpy}" />
+            <inertia ixx="${(m/12) * (3*r*r + l*l)}" ixy="0" ixz="0"
+                     iyy="${(m/12) * (3*r*r + l*l)}" iyz="0"
+                     izz="${(m/2) * (r*r)}" />
         </inertial>
     </xacro:macro>
@@ -28,8 +34,8 @@
         <inertial>
             <mass value="${m}" />
-            <origin xyz="${o_xyz}" rpy="${o_rpy}"/>
-            <inertia ixx="${(2/5) * (m * r * r)}" ixy="0" ixz="0"
-                      iyy="${(2/5) * (m * r * r)}" iyz="0"
-                      izz="${(2/5) * (m * r * r)}" /> <!-- refer to wiki on intertial tensors/moments -->
+            <origin xyz="${o_xyz}" rpy="${o_rpy}" />
+            <inertia ixx="${(2/5) * m * r * r}" ixy="0" ixz="0"
+                     iyy="${(2/5) * m * r * r}" iyz="0"
+                     izz="${(2/5) * m * r * r}" />
         </inertial>
     </xacro:macro>

File: ros2_ws/src/my_robot_description/urdf/mobile_base.xacro (robot description, xacro)
@@ -6,4 +6,22 @@
     <xacro:property name="wheel_radius" value="0.1" />
     <xacro:property name="wheel_length" value="0.05" />
+    <link name="base_footprint" />
+    <link name="base_link">
+        <visual>
+            <geometry>
+                <box size="${base_length} ${base_width} ${base_height}" />
+            </geometry>
+            <origin xyz="0 0 ${base_height / 2.0}" rpy="0 0 0" />
+            <material name="blue" />
+        </visual>
+        <collision>
+            <geometry>
+                <box size="${base_length} ${base_width} ${base_height}" />
+            </geometry>
+            <origin xyz="0 0 ${base_height / 2.0}" rpy="0 0 0" />
+        </collision>
+        <xacro:box_inertia m="5.0" x="${base_length}" y="${base_width}" z="${base_height}"
+                           o_xyz="0 0 ${base_height / 2.0}" o_rpy="0 0 0" />
+    </link>
     <xacro:macro name="wheel_link" params="prefix">
         <link name="${prefix}_wheel_link">
@@ -15,34 +33,16 @@
                 <material name="grey" />
             </visual>
-            <xacro:cylinder_inertia m="5.0" r="${wheel_radius}" h="${wheel_length}"
-                            o_xyz="0 0 0" o_rpy="${pi / 2.0} 0 0"/>
             <collision>
                 <geometry>
                     <sphere radius="${wheel_radius}" />
                 </geometry>
-                <origin xyz="0 0 0" rpy="${pi / 2.0} 0 0" />
+                <origin xyz="0 0 0" rpy="0 0 0" />
             </collision>
+            <xacro:cylinder_inertia m="1.0" r="${wheel_radius}" l="${wheel_length}"
+                                    o_xyz="0 0 0" o_rpy="${pi / 2.0} 0 0" />
         </link>
     </xacro:macro>
     <xacro:wheel_link prefix="right" />
     <xacro:wheel_link prefix="left" />
-    <link name="base_footprint" />
-    <link name="base_link">
-        <visual>
-            <geometry>
-                <box size="${base_length} ${base_width} ${base_height}" /> <!-- LWH in meters -->
-            </geometry>
-            <origin xyz="0 0 ${base_height / 2.0}" rpy="0 0 0" /> <!-- roll pitch yaw - RPY -->
-            <material name="green" />
-        </visual>
-        <xacro:box_inertia m="5.0" x="${base_length}" y="${base_width}" z="${base_height}"
-                            o_xyz="0 0 ${base_height / 2.0}" o_rpy="0 0 0"/>
-         <collision>
-                <geometry>
-                    <box size="${base_length} ${base_width} ${base_height}" />
-                </geometry>
-                <origin xyz="0 0 ${base_height / 2.0}" rpy="0 0 0" />
-        </collision>
-    </link>
     <link name="caster_wheel_link">
         <visual>
@@ -53,22 +53,22 @@
             <material name="grey" />
         </visual>
-        <xacro:sphere_inertia m="5.0" r="${wheel_radius / 2.0}"
-                            o_xyz="0 0 0" o_rpy="0 0 0" />
         <collision>
-                <geometry>
-                    <sphere radius="${wheel_radius / 2.0}" />
-                </geometry>
-                <origin xyz="0 0 0" rpy="0 0 0" />
+            <geometry>
+                <sphere radius="${wheel_radius / 2.0}" />
+            </geometry>
+            <origin xyz="0 0 0" rpy="0 0 0" />
         </collision>
+        <xacro:sphere_inertia m="0.5" r="${wheel_radius / 2.0}"
+                              o_xyz="0 0 0" o_rpy="0 0 0" />
     </link>
     <joint name="base_joint" type="fixed">
         <parent link="base_footprint" />
         <child link="base_link" />
-        <origin xyz="0 0 ${wheel_radius}" rpy="0 0 0" />
+        <origin xyz="0 0 ${wheel_radius}" rpy="0 0 0"/>
     </joint>
     <joint name="base_right_wheel_joint" type="continuous">
         <parent link="base_link" />
         <child link="right_wheel_link" />
-        <origin xyz="${-base_length/4} ${-(base_width + wheel_length ) / 2.0} 0" rpy="0 0 0"/>
+        <origin xyz="${-base_length / 4.0} ${-(base_width + wheel_length) / 2.0} 0" rpy="0 0 0" />
         <axis xyz="0 1 0" />
     </joint>
@@ -76,5 +76,5 @@
         <parent link="base_link" />
         <child link="left_wheel_link" />
-        <origin xyz="${-base_length/4} ${(base_width + wheel_length ) / 2.0} 0" rpy="0 0 0"/>
+        <origin xyz="${-base_length / 4.0} ${(base_width + wheel_length) / 2.0} 0" rpy="0 0 0" />
         <axis xyz="0 1 0" />
     </joint>
@@ -82,5 +82,5 @@
         <parent link="base_link" />
         <child link="caster_wheel_link" />
-        <origin xyz="${base_length/3} 0 ${-wheel_radius / 2.0}" rpy="0 0 0"/>
+        <origin xyz="${base_length / 3.0} 0 ${-wheel_radius / 2.0}" rpy="0 0 0" />
     </joint>
 </robot>

File: ros2_ws/src/my_robot_description/urdf/my_robot.urdf.xacro (robot description, xacro)
@@ -4,4 +4,11 @@
     <xacro:include filename="mobile_base.xacro" />
     <xacro:include filename="mobile_base_gazebo.xacro" />
+    <xacro:include filename="arm.xacro" />
+    <xacro:include filename="arm_gazebo.xacro" />
     <xacro:include filename="camera.xacro" />
+    <joint name="mobile_base_arm_joint" type="fixed">
+        <parent link="base_link" />
+        <child link="arm_base_link" />
+        <origin xyz="${base_length / 4.0} 0 ${base_height}" rpy="0 0 0" />
+    </joint>
 </robot>
